File: wspr_tx_m0_v1/rev-/wspr_tx_m0_v1.kicad_pcb (KiCad board)
At the start: 2 copper layers, 2 parts, among them U1 ATSAMD21G18A-AUT, Y1 Crystal_32k768

Commit message: mass commit, lots of changes to m0 board, not functional yet.  added schematic for featherwinf in PDF form.
Parts:
- added +5V1: +5V, TestPoint:TestPoint_Pad_D1.0mm, F.Cu at (129.5, 109.9)
- added C1: 1uF, digikey-footprints:0805, F.Cu at (139.1, 123.2)
- added C10: C, digikey-footprints:0805, F.Cu at (166.4, 111.8)
- added C11: C, digikey-footprints:0805, F.Cu at (168.9, 111.8)
- added C12: C, digikey-footprints:0805, F.Cu at (170.8, 113.7)
- added C13: C, digikey-footprints:0805, F.Cu at (164.5, 126.4)
- added C14: C, digikey-footprints:0805, F.Cu at (166.4, 124.5)
- added C15: C, digikey-footprints:0805, F.Cu at (168.9, 124.5)
- added C16: C, digikey-footprints:0805, F.Cu at (170.8, 126.4)
- added C17: 1uF, digikey-footprints:0805, F.Cu at (156.8, 124.5)
- added C18: 10uF, digikey-footprints:0805, F.Cu at (135.9, 107.3)
- added C19: 1uF, digikey-footprints:0805, F.Cu at (141.0, 110.5)
- added C2: 1uF, digikey-footprints:0805, F.Cu at (139.1, 121.3)
- added C20: 1uF, digikey-footprints:0805, F.Cu at (141.0, 104.1)
- added C22: 1uF, digikey-footprints:0805, F.Cu at (156.8, 130.8)
- added C23: 1uF, digikey-footprints:0805, F.Cu at (153.7, 127.6)
- added C24: 1uF, digikey-footprints:0805, F.Cu at (137.2, 113.7)
- added C25: 1uF, digikey-footprints:0805, F.Cu at (144.1, 114.3)
- added C3: 22pF, digikey-footprints:0805, F.Cu at (137.2, 116.2)
- added C4: 22pF, digikey-footprints:0805, F.Cu at (137.2, 118.7)
- added C5: 1uF, digikey-footprints:0805, F.Cu at (146.1, 114.3)
- added C6: 1uF, digikey-footprints:0805, F.Cu at (150.5, 114.9)
- added C7: 1uF, digikey-footprints:0805, F.Cu at (146.7, 128.9)
- added C8: 1uF, digikey-footprints:0805, F.Cu at (148.0, 114.3)
- added C9: C, digikey-footprints:0805, F.Cu at (164.5, 113.7)
- added D1: RED, LED_SMD:LED_0805_2012Metric, F.Cu at (130.8, 127.0)
- added D2: GRN, LED_SMD:LED_0805_2012Metric, F.Cu at (130.8, 125.1)
- added DBG1: VREF, TestPoint:TestPoint_Pad_D1.0mm, B.Cu at (151.8, 109.2)
- added DBG2: SWDIO, TestPoint:TestPoint_Pad_D1.0mm, B.Cu at (144.1, 109.2)
- added DBG3: SWCLK, TestPoint:TestPoint_Pad_D1.0mm, B.Cu at (146.7, 109.2)
- added DBG4: GND, TestPoint:TestPoint_Pad_D1.0mm, B.Cu at (149.2, 109.2)
- added F1: Polyfuse, Fuse:Fuse_1206_3216Metric, F.Cu at (133.6, 107.3)
- added H1: MountingHole_Pad, MountingHole:MountingHole_2.2mm_M2_Pad_Via, F.Cu at (129.5, 105.4)
- added H2: MountingHole_Pad, MountingHole:MountingHole_2.2mm_M2_Pad_Via, F.Cu at (129.5, 130.8)
- added H3: MountingHole_Pad, MountingHole:MountingHole_2.2mm_M2_Pad_Via, F.Cu at (175.3, 105.4)
- added H4: MountingHole_Pad, MountingHole:MountingHole_2.2mm_M2_Pad_Via, F.Cu at (175.3, 130.8)
- added J1: RF1, Connector_Coaxial:SMA_Samtec_SMA-J-P-X-ST-EM1_EdgeMount, F.Cu at (175.9, 111.8)
- added J2: RF2, Connector_Coaxial:SMA_Samtec_SMA-J-P-X-ST-EM1_EdgeMount, F.Cu at (175.9, 124.5)
- added J3: USB_B_Micro, Connector_USB:USB_Micro-B_Wuerth_629105150521_CircularHoles, B.Cu at (130.8, 118.1)
- added J4: Conn_01x06_Male, Connector_PinHeader_2.54mm:PinHeader_1x06_P2.54mm_Vertical, F.Cu at (147.3, 105.4)
- added J5: Micro_SD_Card_Det, Connector_Card:microSD_HC_Molex_104031-0811, B.Cu at (146.1, 126.4)
- added L1: L, digikey-footprints:0805, F.Cu at (164.5, 109.9)
- added L2: L, digikey-footprints:0805, F.Cu at (167.6, 108.6)
- added L3: L, digikey-footprints:0805, F.Cu at (170.8, 109.9)
- added L4: L, digikey-footprints:0805, F.Cu at (164.5, 122.6)
- added L5: L, digikey-footprints:0805, F.Cu at (167.6, 121.3)
- added L6: L, digikey-footprints:0805, F.Cu at (170.8, 122.6)
- added R1: 4.7k, digikey-footprints:0805, F.Cu at (155.6, 120.0)
- added R2: 4.7k, digikey-footprints:0805, F.Cu at (153.7, 120.0)
- added R3: 100k, digikey-footprints:0805, F.Cu at (137.8, 107.3)
- added R4: 2.2k, digikey-footprints:0805, F.Cu at (134.6, 127.0)
- added R5: 2.2k, digikey-footprints:0805, F.Cu at (134.6, 125.1)
- added SW1: SW_Push, Button_Switch_SMD:SW_Push_1P1T_NO_CK_KMR2, F.Cu at (154.9, 116.2)
- added U2: Si5351A-B-GT, Package_SO:MSOP-10_3x3mm_P0.5mm, F.Cu at (160.7, 122.6)
- added U3: SPX3819M5-L-3-3, Package_TO_SOT_SMD:SOT-23-5, F.Cu at (141.0, 107.3)
- added U5: MCP9700AT-ELT, Package_TO_SOT_SMD:SOT-353_SC-70-5, F.Cu at (156.2, 127.6)
- added U6: MCP9700AT-ELT, Package_TO_SOT_SMD:SOT-353_SC-70-5, F.Cu at (141.0, 113.0)
- added Y2: Crystal_GND24, Crystal:Crystal_SMD_Abracon_ABM8G-4Pin_3.2x2.5mm, F.Cu at (160.0, 127.6)
- Y1: value Crystal_32k768 -> Crystal; footprint Crystal:Crystal_SMD_Abracon_ABM8G-4Pin_3.2x2.5mm -> Crystal:Crystal_SMD_G8-2Pin_3.2x1.5mm_HandSoldering
- moved Y1 25.0 mm to (140.3, 117.5), turned to 90 degrees
- moved U1 24.1 mm to (146.7, 121.9)
Connections:
- net Net-(U1-Pad10) renamed /A4
- net Net-(U1-Pad12) renamed /D9
- net Net-(U1-Pad14) renamed /D3
- net Net-(U1-Pad15) renamed /D1
- net Net-(U1-Pad16) renamed /D0
- net Net-(U1-Pad23) renamed /D2
- net Net-(U1-Pad24) renamed /D5
- net Net-(U1-Pad25) renamed /D11
- net Net-(U1-Pad27) renamed /D10
- net Net-(U1-Pad28) renamed /D12
- net Net-(U1-Pad29) renamed /D6
- net Net-(U1-Pad37) renamed /TXD
- net Net-(U1-Pad38) renamed /RXD
- net Net-(U1-Pad39) renamed /TXLED
- net Net-(U1-Pad41) renamed /USBHOSTEN
- net Net-(U1-Pad48) renamed /RXLED
- net Net-(U1-Pad7) renamed /A1
- net Net-(U1-Pad8) renamed /A2
- net Net-(U1-Pad9) renamed /A3
- U1 pad 1: EIN1 -> Net-(C3-Pad1)
- U1 pad 11: Net-(U1-Pad11) -> /D8
- U1 pad 13: Net-(U1-Pad13) -> /SD_CS
- U1 pad 17: Net-(U1-Pad17) -> +3V3
- U1 pad 18: Net-(U1-Pad18) -> GND
- U1 pad 19: Net-(U1-Pad19) -> /MOSI
- U1 pad 2: EIN2 -> Net-(C4-Pad1)
- U1 pad 20: Net-(U1-Pad20) -> /SCK
- U1 pad 21: Net-(U1-Pad21) -> /MISO
- U1 pad 26: Net-(U1-Pad26) -> /D13
- U1 pad 3: /MCU/D14_A0 -> /A0
- U1 pad 30: Net-(U1-Pad30) -> /D7
- U1 pad 31: Net-(U1-Pad31) -> /SDA
- U1 pad 32: Net-(U1-Pad32) -> /SCL
- U1 pad 33: Net-(U1-Pad33) -> /D-
- U1 pad 34: Net-(U1-Pad34) -> /D+
- U1 pad 35: Net-(U1-Pad35) -> GND
- U1 pad 36: Net-(U1-Pad36) -> +3V3
- U1 pad 4: /MCU/AREF -> /AREF
- U1 pad 40: Net-(U1-Pad40) -> /~RESET
- U1 pad 42: Net-(U1-Pad42) -> GND
- U1 pad 44: Net-(U1-Pad44) -> +3V3
- U1 pad 45: Net-(U1-Pad45) -> /SWCLK
- U1 pad 46: Net-(U1-Pad46) -> /SWDIO
- U1 pad 47: Net-(U1-Pad47) -> /A5
- U1 pad 5: Net-(U1-Pad5) -> GND
- U1 pad 6: Net-(U1-Pad6) -> +3V3
- Y1 pad 1: EIN1 -> Net-(C4-Pad1)
- Y1 pad 2: GND -> Net-(C3-Pad1)
Routing:
- net +3V3: track 0.00 -> 81.7 mm, vias 0 -> 3
- net /D-: track 0.00 -> 21.6 mm, vias 0 -> 1
- net /D+: track 0.00 -> 20.1 mm, vias 0 -> 1
- net Net-(+5V1-Pad1): track 0.00 -> 18.6 mm, vias 0 -> 1
- net /A0: track 0.00 -> 16.7 mm, vias 0 -> 4
- net /D13: track 0.00 -> 16.1 mm, vias 0 -> 2
- net /SDA: track 0.00 -> 15.7 mm, vias 0 -> 2
- net /SCL: track 0.00 -> 13.4 mm, vias 0 -> 2
- net /LPF Filters/RF2_IN: track 0.00 -> 12.8 mm
- net /D7: track 0.00 -> 12.5 mm, vias 0 -> 1
- net /SWDIO: track 0.00 -> 12.5 mm, vias 0 -> 1
- net /LPF Filters/RF1_IN: track 0.00 -> 12.4 mm
- net /~RESET: track 0.00 -> 11.9 mm, vias 0 -> 2
- net /SWCLK: track 0.00 -> 9.46 mm, vias 0 -> 1
- net /D8: track 0.00 -> 8.05 mm
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- added copper zone on B.Cu, net GND
- added copper zone on F.Cu, net GND
Other:
- board outline added: 50.8 x 30.5 mm
- net class Default: clearance 0.2 -> 0.1524; trace_width 0.25 -> 0.254; via_dia 0.8 -> 0.508; via_drill 0.4 -> 0.254
- rule trace_clearance: 0.2 -> 0.1524
- rule trace_min: 0.2 -> 0.1524
- rule via_min_drill: 0.3 -> 0.254
- rule via_min_size: 0.4 -> 0.508
