File: wspr_tx_m0_v1/rev-/wspr_tx_m0_v1.sch (KiCad schematic (older format))
At the start: 0 parts

Commit message: mass commit, lots of changes to m0 board, not functional yet.  added schematic for featherwinf in PDF form.
Parts:
- added +5V1: +5V, TestPoint:TestPoint_Pad_D1.0mm, symbol Connector:TestPoint
- added C1, C17, C19, C2, C20, C22, C23, C24, C25, C5, C6, C7, C8: 1uF, digikey-footprints:0805, symbol Device:C
- added C18: 10uF, digikey-footprints:0805, symbol Device:C
- added C3, C4: 22pF, digikey-footprints:0805, symbol Device:C
- added D1: RED, LED_SMD:LED_0805_2012Metric, symbol Device:LED
- added D2: GRN, LED_SMD:LED_0805_2012Metric, symbol Device:LED
- added DBG1: VREF, TestPoint:TestPoint_Pad_D1.0mm, symbol Connector:TestPoint
- added DBG2: SWDIO, TestPoint:TestPoint_Pad_D1.0mm, symbol Connector:TestPoint
- added DBG3: SWCLK, TestPoint:TestPoint_Pad_D1.0mm, symbol Connector:TestPoint
- added DBG4: GND, TestPoint:TestPoint_Pad_D1.0mm, symbol Connector:TestPoint
- added F1: Polyfuse, Fuse:Fuse_1206_3216Metric, symbol Device:Polyfuse
- added H1, H2, H3, H4: MountingHole_Pad, MountingHole:MountingHole_2.2mm_M2_Pad_Via, symbol Mechanical:MountingHole_Pad
- added J1: RF1, Connector_Coaxial:SMA_Samtec_SMA-J-P-X-ST-EM1_EdgeMount, symbol Connector:Conn_Coaxial
- added J2: RF2, Connector_Coaxial:SMA_Samtec_SMA-J-P-X-ST-EM1_EdgeMount, symbol Connector:Conn_Coaxial
- added J3: USB_B_Micro, Connector_USB:USB_Micro-B_Wuerth_629105150521_CircularHoles, symbol Connector:USB_B_Micro
- added J4: Conn_01x06_Male, Connector_PinHeader_2.54mm:PinHeader_1x06_P2.54mm_Vertical, symbol Connector:Conn_01x06_Male
- added J5: Micro_SD_Card_Det, Connector_Card:microSD_HC_Molex_104031-0811, symbol Connector:Micro_SD_Card_Det
- added R1, R2: 4.7k, digikey-footprints:0805, symbol Device:R_US
- added R3: 100k, digikey-footprints:0805, symbol Device:R_US
- added R4, R5: 2.2k, digikey-footprints:0805, symbol Device:R_US
- added SW1: SW_Push, Button_Switch_SMD:SW_Push_1P1T_NO_CK_KMR2, symbol Switch:SW_Push
- added U1: ATSAMD21G18A-AUT, digikey-footprints:TQFP-48_7x7mm, symbol dk_Embedded-Microcontrollers:ATSAMD21G18A-AUT
- added U2: Si5351A-B-GT, Package_SO:MSOP-10_3x3mm_P0.5mm, symbol Oscillator:Si5351A-B-GT
- added U3: SPX3819M5-L-3-3, Package_TO_SOT_SMD:SOT-23-5, symbol Regulator_Linear:SPX3819M5-L-3-3
- added U5, U6: MCP9700AT-ELT, Package_TO_SOT_SMD:SOT-353_SC-70-5, symbol Sensor_Temperature:MCP9700AT-ELT
- added Y1: Crystal, Crystal:Crystal_SMD_G8-2Pin_3.2x1.5mm_HandSoldering, symbol Device:Crystal
- added Y2: Crystal_GND24, Crystal:Crystal_SMD_Abracon_ABM8G-4Pin_3.2x2.5mm, symbol Device:Crystal_GND24
Connections:
- new net: C3.1, U1.1 (PA00), Y1.2
- new net: C4.1, U1.2 (PA01), Y1.1
- new net: C8.1, U1.43 (VDDCORE)
- new net: U2.2 (XA), Y2.1
- new net: U2.3 (XB), Y2.3
- new net: +5V1.1, F1.2, J3.1 (VBUS)
- new net: R3.1, U3.3 (EN)
- new net: C19.1, U3.4 (BP)
- new net: D2.2 (A), R5.1
- new net: D1.2 (A), R4.1
- new net +3V3: C1.1, C17.2, C20.1, C22.2, C24.2, C5.1, C6.1, C7.1, DBG1.1, J5.4 (VDD), R1.2, R2.2, U1.17 (VDD/IO), U1.36 (VDD/IO), U1.44 (VDDIN), U1.6 (VDD/ANA), U2.1 (VDD), U2.7 (VDDO), U3.5 (OUT), U5.4 (Vdd), U6.4 (Vdd)
- new net +5V: C18.1, F1.1, R3.2, U3.1 (IN)
- new net A0: C23.2, U1.3 (PA02), U5.3 (Vout)
- new net A1: U1.7 (PB08)
- new net A2: U1.8 (PB09)
- new net A3: U1.9 (PA04)
- new net A4: U1.10 (PA05)
- new net A5: C25.2, U1.47 (PB02), U6.3 (Vout)
- new net AREF: C2.1, U1.4 (PA03)
- new net D+: J3.3 (D+), U1.34 (PA25)
- new net D-: J3.2 (D-), U1.33 (PA24)
- new net D0: U1.16 (PA11)
- new net D1: U1.15 (PA10)
- new net D10: U1.27 (PA18)
- new net D11: U1.25 (PA16)
- new net D12: U1.28 (PA19)
- new net D13: R4.2, U1.26 (PA17)
- new net D2: U1.23 (PA14)
- new net D3: U1.14 (PA09)
- new net D5: U1.24 (PA15)
- new net D6: U1.29 (PA20)
- new net D7: J5.10 (DET_A), U1.30 (PA21)
- new net D8: R5.2, U1.11 (PA06)
- new net D9: U1.12 (PA07)
- new net GND: C1.2, C17.1, C18.2, C19.2, C2.2, C20.2, C22.1, C23.1, C24.1, C25.1, C3.2, C4.2, C5.2, C6.2, C7.2, C8.2, D1.1 (K), D2.1 (K), DBG4.1, H1.1, H2.1, H3.1, H4.1, J1.2 (Ext), J2.2 (Ext), J3.5 (GND), J3.6 (Shield), J5.11 (SHIELD), J5.6 (VSS), SW1.2, U1.18 (GND), U1.35 (GND), U1.42 (GND), U1.5 (GND/ANA), U2.8 (GND), U3.2 (GND), U5.2 (GND), U6.2 (GND), Y2.2, Y2.4
- new net LPF Filters/RF1_IN: U2.10 (CLK0)
- new net LPF Filters/RF1_OUT: J1.1 (In)
- new net LPF Filters/RF2_IN: U2.9 (CLK1)
- new net LPF Filters/RF2_OUT: J2.1 (In)
- new net MISO: J5.7 (DAT0), U1.21 (PA12)
- new net MOSI: J5.3 (CMD), U1.19 (PB10)
- new net RXD: U1.38 (PB23)
- new net RXLED: U1.48 (PB03)
- new net SCK: J5.5 (CLK), U1.20 (PB11)
- new net SCL: R2.1, U1.32 (PA23), U2.4 (SCL)
- new net SDA: R1.1, U1.31 (PA22), U2.5 (SDA)
- new net SD_CS: J5.2 (DAT3/CD), U1.13 (PA08)
- new net SWCLK: DBG3.1, U1.45 (PA30)
- new net SWDIO: DBG2.1, U1.46 (PA31)
- new net TXD: U1.37 (PB22)
- new net TXLED: U1.39 (PA27)
- new net USBHOSTEN: U1.41 (PA28)
- new net ~RESET: SW1.1, U1.40 (~RESET)
